File: huzzashield.kicad_sch (KiCad schematic)
At the start: 10 parts, among them J1 Conn_01x02_Female, J2 Conn_01x04_Female

Commit message: Schematic ad pcb ready
Parts:
- removed R4, R5, R6: R_Small, symbol Device:R_Small
- added J3, J4: Conn_01x01_Female, Connector_PinHeader_2.54mm:PinHeader_1x01_P2.54mm_Vertical, symbol Connector:Conn_01x01_Female
- A1: footprint Module:Adafruit_Feather -> scfablab:FEATHERWING
- D1: footprint (none) -> fabacademy:LED_RGB_Cree_CLV1A-FKB_3.2x2.8mm
- J1: footprint (none) -> sparkfun_connectors:1X02_LONGPADS
- J2: footprint (none) -> sparkfun_connectors:1X04_LONGPADS
- R1, R2, R3: footprint (none) -> Resistor_SMD:R_1206_3216Metric_Pad1.30x1.75mm_HandSolder
Connections:
- net VCC is gone; now on net 3v3: D1.2 (A)
- net GND: now also A1.4 (GND), J1.1 (Pin_1), J2.3 (Pin_3)
- net at R3.1: now also J2.1 (Pin_1)
- net at R3.2: now also A1.15 (TX/IO17)
- net at R2.1: now also J2.2 (Pin_2)
- net at R2.2: now also A1.14 (RX/IO16)
- net 3v3: now reaches A1.2 (3V3)
- net 3v3: now also J2.4 (Pin_4), J3.1 (Pin_1), J4.1 (Pin_1)
- net at A1.21 (A8/IO15): now also D1.4 (GK); no longer D1.3 (BK)
- net at A1.22 (A9/IO33): now also D1.3 (BK); no longer D1.4 (GK)
- net at A1.28 (VBAT): now also J1.2 (Pin_2)
- no-connect marks 0 -> 19
Other:
- moved on the sheet: A1, D1, J1, J2, R1
